File: hardware/autoscreen/autoscreen.kicad_pcb (KiCad board)
At the start: 2 copper layers, 68 x 41 mm, 39 parts, among them J1 USB_B_Micro, J2 Conn_01x06_Male, Q1 Q_Photo_NPN_EC, SW1 SW_Push, SW2 SW_Push, U1 AZ1117-3.3, U2 STM32F722RETx, Y1 12MHz

Commit message: Moved passives away from the TQFP chip for easier rework, and added silkscreen ID
Parts:
- moved R8 1.78 mm to (115.1, 116.2)
- moved R9 1.78 mm to (115.1, 120.7)
- moved C7 0.80 mm to (128.3, 124.0)
- moved C12 0.76 mm to (121.9, 124.0)
Routing:
- net /Vbus: track 117.6 -> 119.6 mm
- net GND: track 124.3 -> 125.5 mm, vias 12 -> 14
- net +3V3: track 126.0 -> 126.7 mm
- net Net-(C7-Pad1): track 3.57 -> 4.23 mm
Other:
- board text added: "AutoScreen"
- board text added: "Rev 1"
